Commit message: update

File: aizo_simulator_description/urdf/falcon4_os1_16_256/falcon4_os1_16_256.gazebo.xacro (robot description, xacro)
@@ -2,4 +2,4 @@
 <robot name="falcon4_os1" xmlns:xacro="http://ros.org/wiki/xacro">
   <xacro:arg name="frame_prefix" default="" />
-  <xacro:include filename="$(find mrsl_quadrotor_description)/urdf/falcon4_os1_16_256/falcon4_os1_16_256.urdf.xacro" frame_prefix="$(arg frame_prefix)"/>
+  <xacro:include filename="$(find aizo_simulator_description)/urdf/falcon4_os1_16_256/falcon4_os1_16_256.urdf.xacro" frame_prefix="$(arg frame_prefix)"/>
 </robot>

File: aizo_simulator_description/urdf/falcon4_os1_16_256/falcon4_os1_16_256.urdf.xacro (robot description, xacro)
@@ -1,5 +1,5 @@
 <?xml version="1.0"?>
 <robot name="quadrotor" xmlns:xacro="http://ros.org/wiki/xacro">
-  <xacro:property name="mass" value="1.8" />
+  <xacro:property name="mass" value="1.2" />
   <xacro:property name="ixx" value="0.004" />
   <xacro:property name="iyy" value="0.004" />
@@ -8,4 +8,5 @@
   <xacro:arg name="robot_ns" default="falcon4"/>
   <xacro:arg name="frame_prefix" default="" />
+  <xacro:arg name="use_nominal_extrinsics" default="true"/>
   <!-- Main quadrotor link -->
   <xacro:macro name="quadrotor_base_macro" params="frame_prefix">
@@ -19,5 +20,5 @@
         <origin xyz="0 0 0.05" rpy="0 0 -${M_PI/2}" />
         <geometry>
-          <mesh filename="package://mrsl_models/models/falcon4/falcon4.dae"/>
+          <mesh filename="package://aizo_models/models/falcon4/falcon4.dae"/>
           <!--cylinder radius="0.05" length="0.01"/-->
         </geometry>
@@ -30,29 +31,59 @@
       </collision>
     </link>
+    <joint name="joint_name" type="fixed">
+      <parent link="base_link"/>
+      <child link="jetson_agx"/>
+      <origin xyz="0 0 0.1" rpy="0 0 0"/>
+      <axis xyz="0 0 1"/>
+    </joint>
+    <link name="jetson_agx">
+      <inertial>
+        <mass value="0.6"/>
+        <origin xyz="-0.03 0.05 0.065" />
+        <inertia ixx="${ixx}" ixy="0.0" ixz="0.0" iyy="${iyy}" iyz="0.0" izz="${izz}" />
+      </inertial>
+      <visual>
+        <origin xyz="-0.03 0.05 0.065" rpy="0 0 -${M_PI/2}" />
+        <geometry>
+          <mesh filename="package://aizo_models/models/jetson_agx/agx.dae" scale="0.001 0.001 0.001"/>
+        </geometry>
+      </visual>
+      <collision>
+        <origin xyz="-0.03 0.05 0.065" rpy="0 0 0" />
+        <geometry>
+          <cylinder radius="0.15" length="0.15"/>
+        </geometry>
+      </collision>
+    </link>
+    <!-- Realme D455 camera -->
+    <xacro:include filename="$(find aizo_simulator_description)/urdf/sensors/realsensed455_camera.urdf.xacro" />
+    <xacro:realsense_camera use_nominal_extrinsics="$(arg use_nominal_extrinsics)" parent="base_link">
+      <origin xyz="0.1 0 0.065" rpy="0 0 0"/>
+    </xacro:realsense_camera>
     <!-- OVC3 Right Side Cam -->
-    <xacro:include filename="$(find mrsl_quadrotor_description)/urdf/sensors/ovc3_extcam.urdf.xacro" />
+    <!-- <xacro:include filename="$(find mrsl_quadrotor_description)/urdf/sensors/ovc3_extcam.urdf.xacro" />
     <xacro:stereo_camera name="bonus_right" parent="base_link" frame_prefix="$(arg frame_prefix)">
       <origin xyz="0.02 -0.084 0.08" rpy="0 0 -${M_PI/2}"/>
-    </xacro:stereo_camera>
+    </xacro:stereo_camera> -->
     <!-- OVC3 Left Side Cam -->
-    <xacro:include filename="$(find mrsl_quadrotor_description)/urdf/sensors/ovc3_extcam.urdf.xacro" />
+    <!-- <xacro:include filename="$(find mrsl_quadrotor_description)/urdf/sensors/ovc3_extcam.urdf.xacro" />
     <xacro:stereo_camera name="bonus_left" parent="base_link" frame_prefix="$(arg frame_prefix)">
       <origin xyz="0.02 0.08 0.08" rpy="0 0 ${M_PI/2}"/>
-    </xacro:stereo_camera>
+    </xacro:stereo_camera> -->
     <!-- OVC3 -->
-    <xacro:include filename="$(find mrsl_quadrotor_description)/urdf/sensors/ovc3.urdf.xacro" />
+    <!-- <xacro:include filename="$(find mrsl_quadrotor_description)/urdf/sensors/ovc3.urdf.xacro" />
     <xacro:stereo_camera name="/ovc3" parent="base_link" frame_prefix="$(arg frame_prefix)">
       <origin xyz="0.1 0 0.065" rpy="0 0 0"/>
-    </xacro:stereo_camera>
+    </xacro:stereo_camera> -->
     <!-- Downward facing Lidar -->
-    <xacro:include filename="$(find mrsl_quadrotor_description)/urdf/sensors/range_beam.urdf.xacro" />
+    <!-- <xacro:include filename="$(find mrsl_quadrotor_description)/urdf/sensors/range_beam.urdf.xacro" />
     <xacro:range_beam name="downward_range_beam_frame" parent="base_link" ros_topic="range" update_rate="10" frame_prefix="$(arg frame_prefix)">
       <origin xyz="0 0 -0.02" rpy="0 ${M_PI/2} 0"/>
-    </xacro:range_beam>
+    </xacro:range_beam>     -->
     <!--Ouster-OS1, hz is frequency, lasers are vertical resolution, samples are horizontal resolution-->
-    <xacro:include filename="$(find mrsl_quadrotor_description)/urdf/sensors/os1-64.urdf.xacro"/>
+    <!-- <xacro:include filename="$(find mrsl_quadrotor_description)/urdf/sensors/os1-64.urdf.xacro"/>
     <xacro:OS1-64 parent="base_link" name="os1_sensor" hz="5" lasers="16" samples="256" robot_ns="$(arg robot_ns)" frame_prefix="$(arg frame_prefix)">
       <origin xyz="0.01 -0.005 0.24" rpy="0 0 0" />
-    </xacro:OS1-64>
+    </xacro:OS1-64> -->
     <!-- Plugins -->
     <gazebo>

File: aizo_simulator_description/urdf/sensors/realsensed455_camera.urdf.xacro (robot description, xacro)
@@ -23,5 +23,5 @@
     <xacro:property name="d455_cam_height" value="0.029"/>
     <xacro:property name="d455_cam_depth" value="0.026"/>
-    <xacro:property name="d455_cam_mount_from_center_offset" value="0.0158"/>
+    <xacro:property name="d455_cam_mount_from_center_offset" value="0.02"/>
     <!-- glass cover is 0.1 mm inwards from front aluminium plate -->
     <xacro:property name="d455_glass_to_front" value="0.1e-3"/>
