Commit message: update

File: aizo_simulator_description/urdf/falcon4_os1_16_256/falcon4_os1_16_256.urdf.xacro (robot description, xacro)
@@ -103,5 +103,5 @@
     </gazebo>
     <!-- GPS Sensor -->
-    <gazebo>
+    <!-- <gazebo>
       <plugin name="novatel_gps_sim" filename="libhector_gazebo_ros_gps.so">
         <alwaysOn>1</alwaysOn>
@@ -115,5 +115,5 @@
           <velocityGaussianNoise>0.1 0.1 0.1</velocityGaussianNoise>
       </plugin>
-    </gazebo>
+    </gazebo> -->
   </xacro:macro>
   <xacro:quadrotor_base_macro frame_prefix="$(arg frame_prefix)"/>

File: aizo_simulator_description/urdf/sensors/realsensed455_camera.urdf.xacro (robot description, xacro)
@@ -6,5 +6,6 @@
 aluminum peripherial evaluation case.
 -->
-<robot name="sensor_d455" xmlns:xacro="http://ros.org/wiki/xacro">
+<robot name="sensor_d455"
+  xmlns:xacro="http://ros.org/wiki/xacro">
   <xacro:property name="M_PI" value="3.1415926535897931" />
   <!-- Includes -->
@@ -54,5 +55,5 @@
         <geometry>
           <!-- <box size="${d455_cam_depth} ${d455_cam_width} ${d455_cam_height}"/> -->
-	        <mesh filename="package://aizo_models//models/sensors/realsense/d455.stl" scale="0.002 0.002 0.002" />
+          <mesh filename="package://aizo_models//models/sensors/realsense/d455.stl" scale="0.002 0.002 0.002" />
         </geometry>
         <material name="aluminum"/>
@@ -129,5 +130,5 @@
       <!-- IMU -->
       <!-- see datasheet Revision 009, page 114 -->
-      <!-- <xacro:property name="d455_imu_px" value="-0.01602"/>
+      <xacro:property name="d455_imu_px" value="-0.01602"/>
       <xacro:property name="d455_imu_py" value="-0.03022"/>
       <xacro:property name="d455_imu_pz" value="+0.0074"/>
@@ -161,11 +162,11 @@
         <parent link="${name}_gyro_optical_frame" />
         <child link="${name}_imu_optical_frame" />
-      </joint> -->
+      </joint>
     </xacro:if>
   </xacro:macro>
   <xacro:macro name="realsense_camera" params=" parent use_nominal_extrinsics *origin">
     <xacro:sensor_d455 parent="${parent}" use_nominal_extrinsics="${use_nominal_extrinsics}">
-        <xacro:insert_block name="origin" />
-      </xacro:sensor_d455>
+      <xacro:insert_block name="origin" />
+    </xacro:sensor_d455>
     <gazebo reference="camera_color_frame">
       <sensor type="depth" name="realsense_R200">
@@ -173,15 +174,15 @@
         <visualize>false</visualize>
         <camera>
-            <horizontal_fov>1.3439</horizontal_fov>
-            <image>
-                <width>640</width>
-                <height>480</height>
-                <format>R8G8B8</format>
-            </image>
-            <depth_camera></depth_camera>
-            <clip>
-                <near>0.03</near>
-                <far>10.0</far>
-            </clip>
+          <horizontal_fov>1.3439</horizontal_fov>
+          <image>
+            <width>640</width>
+            <height>480</height>
+            <format>R8G8B8</format>
+          </image>
+          <depth_camera></depth_camera>
+          <clip>
+            <near>0.03</near>
+            <far>10.0</far>
+          </clip>
         </camera>
         <plugin name="camera_controller" filename="libgazebo_ros_openni_kinect.so">
@@ -198,10 +199,10 @@
           <pointCloudCutoff>0.5</pointCloudCutoff>
           <pointCloudCutoffMax>5.0</pointCloudCutoffMax>
-              <hackBaseline>0.07</hackBaseline>
-              <distortionK1>0.0</distortionK1>
-              <distortionK2>0.0</distortionK2>
-              <distortionK3>0.0</distortionK3>
-              <distortionT1>0.0</distortionT1>
-              <distortionT2>0.0</distortionT2>
+          <hackBaseline>0.07</hackBaseline>
+          <distortionK1>0.0</distortionK1>
+          <distortionK2>0.0</distortionK2>
+          <distortionK3>0.0</distortionK3>
+          <distortionT1>0.0</distortionT1>
+          <distortionT2>0.0</distortionT2>
           <CxPrime>0.0</CxPrime>
           <Cx>0.0</Cx>
@@ -212,4 +213,23 @@
       </sensor>
     </gazebo>
+    <gazebo reference="camera_link">
+      <gravity>true</gravity>
+      <sensor name="imu_sensor" type="imu">
+        <always_on>true</always_on>
+        <update_rate>100</update_rate>
+        <visualize>true</visualize>
+        <plugin filename="libgazebo_ros_imu_sensor.so" name="imu_plugin">
+          <topicName>imu/data_raw</topicName>
+          <bodyName>camera_link</bodyName>
+          <updateRateHZ>10.0</updateRateHZ>
+          <gaussianNoise>0.0</gaussianNoise>
+          <xyzOffset>0 0 0</xyzOffset>
+          <rpyOffset>0 0 0</rpyOffset>
+          <frameName>camera_link</frameName>
+          <initialOrientationAsReference>false</initialOrientationAsReference>
+        </plugin>
+        <pose>0 0 0 0 0 0</pose>
+      </sensor>
+    </gazebo>
   </xacro:macro>
 </robot>
